File: vb124_iob_isofd_db9/vb124_iob_isofd_db9.kicad_pcb (KiCad board)
At the start: 2 copper layers, 33 parts, among them M1 B0505MT-1WR4, Q1 FDN358P, Q2 FDN358P, SW1 DS04-254-2-03BK-SMT, U1 ADM3057E, U2 LAN8740A, U2 STM32H725IGK6

Commit message: vb124
Parts:
- removed U2: STM32H725IGK6, _Test_Library:UFBGA-201_10x10mm_Layout15x15_P0.65mm
- removed U2: LAN8740A, vhrd_interface_ethernet:QFN-32-1EP_5x5mm_P0.5mm_EP3.3x3.3mm_ThermalVias
- added M2: iob_v2, vhrd_module_custom:iob_v2_module, F.Cu at (178.8, 96.5)
- moved U1 62.9 mm to (200.7, 114.3), turned to 90 degrees
- moved M1 48.4 mm to (188.0, 114.3)
Other:
- board outline added: 32 x 35 mm
