File: vb125_eth_fdcan_pro/p10_block_diagram.kicad_sch (KiCad schematic)
At the start: 0 parts

Commit message: Add testpoints and set page templates.
Other:
- company: (none) -> vhrd.tech AS
- title: (none) -> rt_bridge_pro
Changed lines of the file:
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@@
 (kicad_sch (version 20230121) (generator eeschema)
-  (paper "A4")
+  (paper "A3")
+  (title_block
+    (title "rt_bridge_pro")
+    (date "2023-04-21")
+    (rev "A")
+    (company "vhrd.tech AS")
+    (comment 1 "Isaikin R.E.")
+    (comment 4 "Draft")
+  )
 )
