File: vb125_eth_fdcan_pro/p11_mechanical.kicad_sch (KiCad schematic)
At the start: 4 parts

Commit message: Add testpoints and set page templates.
Other:
- company: (none) -> vhrd.tech AS
- title: (none) -> rt_bridge_pro
Changed lines of the file:
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@@
 (kicad_sch (version 20230121) (generator eeschema)
-  (paper "A4")
+  (paper "A3")
+  (title_block
+    (title "rt_bridge_pro")
+    (date "2023-04-21")
+    (rev "A")
+    (company "vhrd.tech AS")
+    (comment 1 "Isaikin R.E.")
+    (comment 4 "Draft")
+  )
   (wire (pts (xy 53.34 38.1) (xy 53.34 40.64))
     (stroke (width 0) (type default))
@@
         )
         (path "/b473bccb-f14c-41d5-b473-137d3ef8ae1e/26a60099-c518-4417-8985-d5c8399fcac3"
-          (reference "#PWR0171") (unit 1)
+          (reference "#PWR0199") (unit 1)
         )
       )
@@
         )
         (path "/b473bccb-f14c-41d5-b473-137d3ef8ae1e/26a60099-c518-4417-8985-d5c8399fcac3"
-          (reference "#PWR0172") (unit 1)
+          (reference "#PWR0200") (unit 1)
         )
       )
@@
         )
         (path "/b473bccb-f14c-41d5-b473-137d3ef8ae1e/26a60099-c518-4417-8985-d5c8399fcac3"
-          (reference "#PWR0169") (unit 1)
+          (reference "#PWR0197") (unit 1)
         )
       )
@@
         )
         (path "/b473bccb-f14c-41d5-b473-137d3ef8ae1e/26a60099-c518-4417-8985-d5c8399fcac3"
-          (reference "#PWR0170") (unit 1)
-        )
-      )
+          (reference "#PWR0198") (unit 1)
+        )
+      )
