File: vb125_eth_fdcan_pro/p2_mcu_h7.kicad_sch (KiCad schematic)
At the start: 63 parts, among them J1 MEM2061-01-188-00-A, J2 TAGconnect NL, J3 Conn_02x20_Pin, M1 DM-OLED042-647, U1 STM32H725IGKx, X1 ECX-.327-CDX-1293

Commit message: Finish layout.
Parts:
- removed J3: Conn_02x20_Pin, Connector_PinHeader_1.27mm:PinHeader_2x20_P1.27mm_Vertical_SMD, symbol vhrd_connector_generic:Conn_02x20_Pin
- removed R9 (x2): 3K3, Resistor_SMD:R_0402_1005Metric, symbol Device:R
- added TP46, TP47, TP48, TP49: TestPoint_Probe, TestPoint:TestPoint_Pad_D1.5mm, symbol Connector:TestPoint_Probe
- added TP50, TP51, TP52, TP53, TP54: TestPoint, TestPoint:TestPoint_Pad_D1.0mm, symbol Connector:TestPoint
Connections:
- net BOOT0: now also TP49.1
- net BUTTON: now also U1.R12 (PE11); no longer U1.F15 (PG5)
- net GND: now also TP51.1
- net H7_SWCLK: now also TP47.1
- net H7_SWDIO: now also TP46.1
- net OLED_RST: now also U1.R3 (PA0_C); no longer U1.G3 (PF2)
- net RID_BOM: now also U1.R10 (PF14); no longer U1.N7 (PF11)
- net RID_EN: now also U1.P13 (PE13); no longer U1.P5 (PA4)
- net RID_PRODUCT: now also U1.P11 (PF12); no longer U1.P3 (PA1_C)
- net RID_REV: now also U1.N11 (PF13); no longer U1.R7 (PA6)
- net RJ45_LEDG: now also U1.H2 (PF4); no longer U1.G15 (PG2)
- net RJ45_LEDY: now also U1.H3 (PF5); no longer U1.H13 (PG3)
- net SPI1_MISO: now also TP52.1
- net SPI1_MOSI: now also TP53.1
- net SPI1_NSS: now also TP54.1
- net SPI1_SCK: now also TP50.1
- net TERM1_DIS: now also U1.B1 (PE4); no longer U1.K13 (PD9)
- net TERM1_EN: now also U1.C1 (PC13); no longer U1.L14 (PD8)
- net TERM2_DIS: now also U1.C14 (PA10); no longer U1.G12 (PG8)
- net TERM2_EN: now also U1.B14 (PA8); no longer U1.G13 (PG7)
- net ULPI_RST: now also U1.R4 (PH3); no longer U1.D8 (PG12)
- net ~{ETH_PHY_RST}: now also U1.N2 (PC3_C); no longer U1.N9 (PG1)
- net ~{H7_RST}: now also TP48.1
- net USBFS_DM renamed USBFS_D_N
- net USBFS_DP renamed USBFS_D_P
- no-connect marks 57 -> 56
Other:
- note added: "Expansion points"
- note removed: "Expansion port"
