File: vb125_eth_fdcan_pro/vb125_eth_fdcan_pro.kicad_pcb (KiCad board)
At the start: 4 copper layers, 105 x 82 mm, 333 parts, among them J1 MEM2061-01-188-00-A, J2 TAGconnect NL, J3 Conn_02x20_Pin, J4 ARJM11D7-114-AB, J5 USB_C_Receptacle_USB2.0, J6 D09P33E4GL00LF, J7 D09P33E4GL00LF, K1 EE2-4.5TNUH, K2 EE2-4.5TNUH, M1 DM-OLED042-647, M2 B0505MT-1WR4, M3 B0505MT-1WR4, Q1 BSS138, Q2 BSS138, Q3 BSS138, Q4 BSS138, Q5 MMBTA42, Q6 Si3440DV, Q7 2N7002, SW1 KSS331GLFS, T1 PA1134NL, T2 750315125, U1 STM32H725IGKx, U10 TLP2270, U11 LTC4267, U12 PS2911-1-F3-AX, U13 ZR431, U14 LV14360SDDAR, U15 LT8304IS8E#PBF, U2 LAN8740A, U3 NCP563SQ18T1G, U4 USB3315, U5 AOZ1376DI-02, U6 RT5760A/B, U7 ADM3050EBRIZ, U8 TLP2270, U9 ADM3050EBRIZ, X1 ECX-.327-CDX-1293, X2 50MHz, X3 24MHz

Commit message: Floorplan work.
Parts:
- removed C103: 10uF, Capacitor_SMD:C_1210_3225Metric
- removed C105, C107, C109: 100nF, Capacitor_SMD:C_0402_1005Metric
- removed C111: 100uF, Capacitor_SMD:C_1210_3225Metric
- removed D21: PDS360-13, Diode_SMD:D_PowerDI-5
- removed JP1: Jumper board, vhrd_generic:PCB_JUMPER
- removed L6: LMLP07A7M8R2DTAS, vhrd_inductor:LMLP07A7
- removed R88: 49K9, Resistor_SMD:R_0402_1005Metric
- removed R91, R97: 10K, Resistor_SMD:R_0402_1005Metric
- removed R96: 57K6, Resistor_SMD:R_0402_1005Metric
- removed TP37: TestPoint_Probe, TestPoint:TestPoint_Pad_D1.5mm
- removed U14: LV14360SDDAR, Package_SO:SOIC-8-1EP_3.9x4.9mm_P1.27mm_EP2.95x4.9mm_Mask2.71x3.4mm_ThermalVias
- J1: moved to F.Cu
- TP1, TP10, TP11, TP12, TP13, TP14, TP15, TP16, TP17, TP18, TP19, TP2, TP20, TP21, TP22, TP23, TP24, TP25, TP26, TP27, TP28, TP29, TP3, TP30, TP31, TP32, TP33, TP34, TP35, TP36, TP38, TP39, TP4, TP40, TP5, TP6, TP7, TP8, TP9: moved to B.Cu
- moved C64 116.3 mm to (151.0, 118.2)
- moved FB3 116.3 mm to (151.0, 120.7)
- moved C62 116.3 mm to (151.0, 115.7)
- moved C76 106.1 mm to (151.7, 127.3)
- moved C78 106.1 mm to (151.7, 129.8)
- moved FB5 106.1 mm to (151.7, 132.3)
- moved C61 92.3 mm to (159.0, 121.4)
- moved C63 92.3 mm to (159.0, 123.4)
- moved C60 86.2 mm to (155.2, 118.9)
- moved C59 86.2 mm to (155.2, 115.9)
- moved C75 82.0 mm to (159.7, 133.0)
- moved C77 82.0 mm to (159.7, 135.0)
- moved C74 79.6 mm to (155.9, 130.5)
- moved C73 79.6 mm to (155.9, 127.5)
- moved L3 77.8 mm to (155.3, 121.8)
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Connections:
- net Net-(C64-Pad1) renamed /CAN Ch1/+5V0_MFLT
- net Net-(C78-Pad1) renamed /CAN Ch2/+5V0_MFLT

Commit message: Continue with floorplan
Parts:
- C10, C11, C12, C13, C14, C16, C19, C21, C22, C23, C24, C26, C27, C28, FB1: moved to F.Cu
- moved R15 84.3 mm to (132.2, 165.5)
- moved L3 41.0 mm to (161.5, 81.2)
- moved C62 37.6 mm to (161.5, 79.6)
- moved C64 36.8 mm to (161.5, 82.9), turned to 180 degrees
- moved C55 33.8 mm to (119.7, 97.0), turned to -90 degrees
- moved C56 29.6 mm to (119.2, 94.3), turned to 90 degrees
- moved C52 26.9 mm to (112.3, 95.7), turned to 180 degrees
- moved U6 26.7 mm to (116.2, 98.5), turned to -90 degrees
- moved R3 25.1 mm to (141.8, 109.2)
- moved C63 24.1 mm to (162.0, 99.5), turned to 180 degrees
- moved L4 23.7 mm to (161.2, 110.2)
- moved R4 23.7 mm to (134.7, 105.5), turned to 180 degrees
- moved R61 23.3 mm to (161.2, 92.2)
- moved C78 23.2 mm to (161.3, 108.6), turned to 180 degrees
- moved R6 22.0 mm to (134.8, 100.5), turned to 0 degrees
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
Commit message: Continue with floorplan
Parts:
- removed SW1: KSS331GLFS, vhrd_electromechanical:SW_KSS3
- added VB125C1: vb125c1_button_board, vhrd_boards:vb125c1_button_board, F.Cu at (118.8, 108.5)
- moved Q6 66.8 mm to (125.8, 67.9), turned to 0 degrees
- moved C92 62.3 mm to (142.7, 77.8)
- moved Q7 62.0 mm to (138.9, 74.2), turned to 180 degrees
- moved R80 55.7 mm to (138.7, 80.0)
- moved R78 55.5 mm to (132.6, 80.1), turned to 180 degrees
- moved R69 54.3 mm to (135.9, 75.0), turned to 180 degrees
- moved R75 53.3 mm to (138.7, 78.0), turned to 180 degrees
- moved R81 52.7 mm to (135.9, 80.0), turned to 180 degrees
- moved R76 52.5 mm to (138.7, 79.0), turned to 180 degrees
- moved R72 49.9 mm to (135.9, 76.0), turned to 180 degrees
- moved R70 49.1 mm to (132.6, 72.9)
- moved D13 48.3 mm to (135.9, 78.7)
- moved D14 47.3 mm to (138.7, 76.8)
- moved R71 47.0 mm to (127.8, 74.7)
- moved C93 46.1 mm to (145.1, 80.5)
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
Commit message: Update vb125_eth_fdcan_pro.kicad_pcb
Parts:
- moved R67 79.8 mm to (177.6, 132.7)
- moved FB6 79.6 mm to (177.6, 110.6), turned to -90 degrees
- moved Q3 74.4 mm to (181.3, 114.1), turned to -90 degrees
- moved D6 73.7 mm to (183.9, 114.7), turned to -90 degrees
- moved C83 70.2 mm to (175.8, 110.6), turned to -90 degrees
- moved R68 69.9 mm to (186.9, 120.9), turned to -90 degrees
- moved C85 69.7 mm to (176.6, 113.4), turned to 180 degrees
- moved D7 69.6 mm to (186.9, 129.9), turned to 90 degrees
- moved Q4 68.2 mm to (181.4, 133.9), turned to 90 degrees
- moved C86 61.1 mm to (186.9, 125.2), turned to -90 degrees
- moved R56 40.2 mm to (122.4, 93.9)
- moved R55 40.1 mm to (122.4, 92.9)
- moved R57 37.8 mm to (119.8, 93.4)
- moved R59 36.2 mm to (118.3, 98.7)
- moved R58 36.0 mm to (118.3, 99.7)
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
Commit message: Finish layout.
Parts:
- removed C39: 100nF, Capacitor_SMD:C_0402_1005Metric
- removed J3: Conn_02x20_Pin, Connector_PinHeader_1.27mm:PinHeader_2x20_P1.27mm_Vertical_SMD
- removed R3, R4: 3K3, Resistor_SMD:R_0402_1005Metric
- removed TP30, TP38, TP39: TestPoint_Probe, TestPoint:TestPoint_Pad_D1.5mm
- added D16: RCLAMP0502BA, Package_TO_SOT_SMD:SOT-416, F.Cu at (106.7, 93.6)
- added D21: RCLAMP0502BA, Package_TO_SOT_SMD:SOT-416, F.Cu at (120.9, 73.1)
- added TP37: TestPoint_Probe, TestPoint:TestPoint_Pad_D1.5mm, B.Cu at (184.8, 74.3)
- added TP42: TestPoint_Probe, TestPoint:TestPoint_Pad_D1.5mm, B.Cu at (106.7, 91.3)
- added TP46: TestPoint_Probe, TestPoint:TestPoint_Pad_D1.5mm, B.Cu at (115.1, 122.3)
- added TP47: TestPoint_Probe, TestPoint:TestPoint_Pad_D1.5mm, B.Cu at (115.0, 124.9)
- added TP48: TestPoint_Probe, TestPoint:TestPoint_Pad_D1.5mm, B.Cu at (120.3, 121.1)
- added TP49: TestPoint_Probe, TestPoint:TestPoint_Pad_D1.5mm, B.Cu at (120.3, 123.7)
- added TP50: TestPoint, TestPoint:TestPoint_Pad_D1.0mm, B.Cu at (146.9, 105.8)
- added TP51: TestPoint, TestPoint:TestPoint_Pad_D1.0mm, B.Cu at (148.5, 105.3)
- added TP52: TestPoint, TestPoint:TestPoint_Pad_D1.0mm, B.Cu at (145.9, 104.5)
- added TP53: TestPoint, TestPoint:TestPoint_Pad_D1.0mm, B.Cu at (145.3, 107.8)
- added TP54: TestPoint, TestPoint:TestPoint_Pad_D1.0mm, B.Cu at (145.3, 109.0)
- D1: value D5V0P4UR6SO-7 -> RCLAMP0502BA; footprint vhrd_passive_tvs:D5V0P4UR6SO-7 -> Package_TO_SOT_SMD:SOT-416
- moved TP10 117.2 mm to (150.9, 108.0)
- moved TP20 115.0 mm to (165.9, 113.7)
- moved TP3 114.0 mm to (141.4, 98.5)
- moved TP23 113.4 mm to (130.9, 60.8)
- moved TP16 113.3 mm to (165.6, 86.1)
- moved TP19 110.9 mm to (168.9, 116.8)
- moved TP15 109.5 mm to (169.9, 86.8)
- moved TP27 105.6 mm to (122.4, 68.9)
- moved TP21 101.8 mm to (179.7, 115.5), turned to -90 degrees
- moved TP22 101.8 mm to (179.7, 119.2), turned to -90 degrees
- moved TP18 98.9 mm to (179.7, 84.6)
- moved TP17 98.9 mm to (179.7, 80.9)
- moved TP2 95.8 mm to (110.3, 127.0)
- moved TP1 95.7 mm to (107.0, 127.0)
- moved C79 95.3 mm to (157.5, 134.4)
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Connections:
- net /USB/DM renamed /USB/D_N
- net /USB/DP renamed /USB/D_P
- net USBFS_DM renamed USBFS_D_N
- net USBFS_DP renamed USBFS_D_P
- D1 pad 1: /Eth/RD- -> /Eth/RD_P
- D1 pad 2: GND -> /Eth/RD_N
- D1 pad 3: /Eth/TD- -> CHASSIS
- J4 pad 10: /Eth/TD+ -> /Eth/TD_P
- J4 pad 3: /Eth/RD- -> /Eth/RD_N
- J4 pad 5: /Eth/RD+ -> /Eth/RD_P
- J4 pad 8: /Eth/TD- -> /Eth/TD_N
- J6 pad 1: /Bus Power/+VIN_DB9 -> unconnected-(J6-Pad1)
- J7 pad 1: /CAN Ch2/+VIN_DB9 -> unconnected-(J7-Pad1)
- K1 pad 4: Net-(C72-Pad1) -> Net-(K1-Pad4)
- K1 pad 5: Net-(K1-Pad5) -> /CAN Ch1/CAN_H
- K1 pad 8: Net-(K1-Pad8) -> /CAN Ch1/CAN_L
- K1 pad 9: Net-(C72-Pad1) -> Net-(K1-Pad9)
- K2 pad 4: Net-(C86-Pad1) -> Net-(K2-Pad4)
- K2 pad 5: Net-(K2-Pad5) -> /CAN Ch2/CAN_H
- K2 pad 8: Net-(K2-Pad8) -> /CAN Ch2/CAN_L
- K2 pad 9: Net-(C86-Pad1) -> Net-(K2-Pad9)
- R35 pad 2: /Eth/RD- -> /Eth/RD_N
- R36 pad 2: /Eth/RD+ -> /Eth/RD_P
- R38 pad 2: /Eth/TD- -> /Eth/TD_N
- R39 pad 2: /Eth/TD+ -> /Eth/TD_P
- R63 pad 1: /CAN Ch1/CAN_H -> Net-(K1-Pad4)
- R63 pad 2: Net-(K1-Pad5) -> Net-(C72-Pad1)
- R64 pad 1: /CAN Ch1/CAN_L -> Net-(K1-Pad9)
- R64 pad 2: Net-(K1-Pad8) -> Net-(C72-Pad1)
- R67 pad 1: /CAN Ch2/CAN_H -> Net-(K2-Pad4)
- R67 pad 2: Net-(K2-Pad5) -> Net-(C86-Pad1)
- R68 pad 1: /CAN Ch2/CAN_L -> Net-(K2-Pad9)
- R68 pad 2: Net-(K2-Pad8) -> Net-(C86-Pad1)
- U1 pad A10: /CAN Ch2/FDCAN_TX -> /CAN Ch1/FDCAN_TX
- U1 pad A2: /CAN Ch2/FDCAN_RX -> /CAN Ch1/FDCAN_RX
- U1 pad A8: /CAN Ch1/FDCAN_TX -> /CAN Ch2/FDCAN_TX
- U1 pad B1: unconnected-(U1E-PE4-PadB1) -> /CAN Ch1/TERM_DIS
- U1 pad B14: unconnected-(U1A-PA8-PadB14) -> /CAN Ch2/TERM_EN
- U1 pad C1: unconnected-(U1C-PC13-PadC1) -> /CAN Ch1/TERM_EN
- U1 pad C14: unconnected-(U1A-PA10-PadC14) -> /CAN Ch2/TERM_DIS
- U1 pad C8: /CAN Ch1/FDCAN_RX -> /CAN Ch2/FDCAN_RX
- U1 pad D8: ULPI_RST -> unconnected-(U1G-PG12-PadD8)
- U1 pad F15: /MCU_H7/BUTTON -> unconnected-(U1G-PG5-PadF15)
- U1 pad G12: /CAN Ch1/TERM_DIS -> unconnected-(U1G-PG8-PadG12)
- U1 pad G13: /CAN Ch1/TERM_EN -> unconnected-(U1G-PG7-PadG13)
- U1 pad G15: RJ45_LEDG -> unconnected-(U1G-PG2-PadG15)
- U1 pad G3: /MCU_H7/OLED_RST -> unconnected-(U1F-PF2-PadG3)
- U1 pad H13: RJ45_LEDY -> unconnected-(U1G-PG3-PadH13)
- U1 pad H2: unconnected-(U1F-PF4-PadH2) -> RJ45_LEDG
- U1 pad H3: unconnected-(U1F-PF5-PadH3) -> RJ45_LEDY
- U1 pad K13: /CAN Ch2/TERM_DIS -> unconnected-(U1D-PD9-PadK13)
- U1 pad L14: /CAN Ch2/TERM_EN -> unconnected-(U1D-PD8-PadL14)
- U1 pad N11: unconnected-(U1F-PF13-PadN11) -> /MCU_H7/RID_REV
- U1 pad N2: unconnected-(U1C-PC3_C-PadN2) -> ~{ETH_PHY_RST}
- U1 pad N7: /MCU_H7/RID_BOM -> unconnected-(U1F-PF11-PadN7)
- U1 pad N9: ~{ETH_PHY_RST} -> unconnected-(U1G-PG1-PadN9)
- U1 pad P11: unconnected-(U1F-PF12-PadP11) -> /MCU_H7/RID_PRODUCT
- U1 pad P13: unconnected-(U1E-PE13-PadP13) -> /MCU_H7/RID_EN
- U1 pad P3: /MCU_H7/RID_PRODUCT -> unconnected-(U1A-PA1_C-PadP3)
- U1 pad P5: /MCU_H7/RID_EN -> unconnected-(U1A-PA4-PadP5)
- U1 pad R10: unconnected-(U1F-PF14-PadR10) -> /MCU_H7/RID_BOM
- U1 pad R12: unconnected-(U1E-PE11-PadR12) -> /MCU_H7/BUTTON
- U1 pad R3: unconnected-(U1A-PA0_C-PadR3) -> /MCU_H7/OLED_RST
- U1 pad R4: unconnected-(U1H-PH3-PadR4) -> ULPI_RST
- U1 pad R7: /MCU_H7/RID_REV -> unconnected-(U1A-PA6-PadR7)
- U2 pad 28: /Eth/TD- -> /Eth/TD_N
- U2 pad 29: /Eth/TD+ -> /Eth/TD_P
- U2 pad 30: /Eth/RD- -> /Eth/RD_N
- U2 pad 31: /Eth/RD+ -> /Eth/RD_P
Routing:
- net GND: track 0.00 -> 157.9 mm, vias 0 -> 186
- net +3V3_DCDC: track 0.00 -> 80.0 mm, vias 0 -> 55
- net /MCU_H7/VBAT: track 0.00 -> 62.0 mm, vias 0 -> 2
- net /Eth/+AVDD_PHY: track 0.00 -> 57.9 mm, vias 0 -> 6
- net /MCU_H7/~{H7_RST}: track 0.00 -> 51.4 mm, vias 0 -> 4
- net /MCU_H7/SDMMC_D1: track 0.00 -> 50.3 mm
- net /MCU_H7/I2C2_SDA: track 0.00 -> 50.0 mm, vias 0 -> 2
- net /MCU_H7/SDMMC_D0: track 0.00 -> 50.0 mm
- net /MCU_H7/SDMMC_CMD: track 0.00 -> 48.7 mm, vias 0 -> 2
- net /MCU_H7/I2C2_SCL: track 0.00 -> 48.1 mm, vias 0 -> 2
- net /MCU_H7/SDMMC_D2: track 0.00 -> 47.6 mm, vias 0 -> 2
- net /MCU_H7/SDMMC_D3: track 0.00 -> 47.6 mm, vias 0 -> 2
- net /MCU_H7/SDMMC_CK: track 0.00 -> 45.5 mm, vias 0 -> 2
- net /MCU_H7/BOOT0: track 0.00 -> 44.2 mm, vias 0 -> 3
- net RJ45_LEDG: track 0.00 -> 43.0 mm, vias 0 -> 2
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- added copper zone on F.Cu, net +3V3_DCDC
- added copper zone on In4.Cu, net +3V3_DCDC
- added copper zone on F.Cu, net +5V0_SYS
- added copper zone on In3.Cu, net +5V0_SYS
- added copper zone on B.Cu, net +VIN_USB
- added copper zone on F.Cu, net +VIN_USB
- added copper zone on F.Cu, net /Bus Power/+VIN_DB9
- added copper zone on F.Cu, net /Bus Power/+VIN_DB9_PR
- added copper zone on F.Cu, net /Bus Power/RECT_COMMON
- added copper zone on F.Cu, net /CAN Ch1/+5V0_ISO
- added copper zone on In2.Cu, net /CAN Ch1/+5V0_ISO
- added copper zone on F.Cu, net /CAN Ch1/+VO
- added copper zone on F.Cu, net /CAN Ch2/+5V0_ISO
- added copper zone on In2.Cu, net /CAN Ch2/+5V0_ISO
- added copper zone on F.Cu, net /CAN Ch2/+VO
- added copper zone on F.Cu, net /CAN Ch2/ISO
- added copper zone on In1.Cu, net /CAN Ch2/ISO
- added copper zone on In3.Cu, net /MCU_H7/VDDA
- added copper zone on F.Cu, net /MCU_H7/VDDLDO
- added copper zone on In3.Cu, net /MCU_H7/VDDLDO
- added copper zone on F.Cu, net /PoE/POE_BR_N
- added copper zone on In3.Cu, net /PoE/POE_BR_N
- added copper zone on F.Cu, net /PoE/POE_BR_P
- added copper zone on B.Cu, net /PoE/POE_EP_THPAD
- added copper zone on In2.Cu, net /PoE/POE_EP_THPAD
- added copper zone on F.Cu, net /PoE/POE_VPORTP
- added copper zone on In2.Cu, net /PoE/POE_VPORTP
- added copper zone on F.Cu, net /Power/3V3_SW
- added copper zone on B.Cu, net CHASSIS
- added copper zone on F.Cu, net CHASSIS
- added copper zone on In1.Cu, net CHASSIS
- added copper zone on In2.Cu, net CHASSIS
- added copper zone on In3.Cu, net CHASSIS
- added copper zone on In4.Cu, net CHASSIS
- added copper zone on F.Cu, net GND
- added copper zone on In1.Cu, net GND
- added copper zone on In3.Cu, net GND
- added copper zone on In4.Cu, net GND
- added copper zone on F.Cu, net ISO_1
- added copper zone on In1.Cu, net ISO_1
- added copper zone on F.Cu, net ISO_POE
- added copper zone on In1.Cu, net ISO_POE
- added copper zone on In4.Cu, net ISO_POE
Other:
- board size 105 x 82 mm -> 96 x 82 mm
- copper layers 4 -> 6
