File: vb125_eth_fdcan_pro/vb125_eth_fdcan_pro.kicad_sch (KiCad schematic)
At the start: 0 parts

Commit message: Finish layout.
Parts:
- added TP1: TestPoint_Probe, TestPoint:TestPoint_Pad_D1.5mm, symbol Connector:TestPoint_Probe
Connections:
- net Bus Power/+VIN_DB9: now also TP1.1
Changed lines of the file:
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@@
     (comment 4 "Draft")
   )
+  (junction (at 212.09 142.24) (diameter 0) (color 0 0 0 0)
+  )
   (wire (pts (xy 209.55 148.59) (xy 205.74 148.59))
     (stroke (width 0) (type default))
   )
+  (wire (pts (xy 209.55 151.13) (xy 209.55 148.59))
+    (stroke (width 0) (type default))
+  )
+  (wire (pts (xy 251.46 157.48) (xy 251.46 142.24))
+    (stroke (width 0) (type default))
+  )
+  (wire (pts (xy 166.37 119.38) (xy 173.99 119.38))
+    (stroke (width 0) (type default))
+  )
   (wire (pts (xy 166.37 125.73) (xy 173.99 125.73))
     (stroke (width 0) (type default))
   )
-  (wire (pts (xy 209.55 151.13) (xy 209.55 148.59))
-    (stroke (width 0) (type default))
-  )
-  (wire (pts (xy 251.46 157.48) (xy 251.46 142.24))
+  (wire (pts (xy 251.46 142.24) (xy 248.92 142.24))
+    (stroke (width 0) (type default))
+  )
+  (wire (pts (xy 166.37 121.92) (xy 173.99 121.92))
+    (stroke (width 0) (type default))
+  )
+  (wire (pts (xy 205.74 142.24) (xy 212.09 142.24))
+    (stroke (width 0) (type default))
+  )
+  (wire (pts (xy 248.92 157.48) (xy 251.46 157.48))
+    (stroke (width 0) (type default))
+  )
+  (wire (pts (xy 166.37 149.86) (xy 173.99 149.86))
+    (stroke (width 0) (type default))
+  )
+  (wire (pts (xy 212.09 142.24) (xy 217.17 142.24))
+    (stroke (width 0) (type default))
+  )
+  (wire (pts (xy 166.37 147.32) (xy 173.99 147.32))
+    (stroke (width 0) (type default))
+  )
+  (wire (pts (xy 166.37 143.51) (xy 173.99 143.51))
+    (stroke (width 0) (type default))
+  )
+  (wire (pts (xy 212.09 138.43) (xy 212.09 142.24))
+    (stroke (width 0) (type default))
+  )
+  (wire (pts (xy 166.37 140.97) (xy 173.99 140.97))
     (stroke (width 0) (type default))
   )
   (wire (pts (xy 166.37 128.27) (xy 173.99 128.27))
-    (stroke (width 0) (type default))
-  )
-  (wire (pts (xy 166.37 147.32) (xy 173.99 147.32))
-    (stroke (width 0) (type default))
-  )
-  (wire (pts (xy 251.46 142.24) (xy 248.92 142.24))
-    (stroke (width 0) (type default))
-  )
-  (wire (pts (xy 166.37 149.86) (xy 173.99 149.86))
-    (stroke (width 0) (type default))
-  )
-  (wire (pts (xy 205.74 142.24) (xy 217.17 142.24))
-    (stroke (width 0) (type default))
-  )
-  (wire (pts (xy 248.92 157.48) (xy 251.46 157.48))
-    (stroke (width 0) (type default))
-  )
-  (wire (pts (xy 166.37 140.97) (xy 173.99 140.97))
-    (stroke (width 0) (type default))
-  )
-  (wire (pts (xy 166.37 119.38) (xy 173.99 119.38))
-    (stroke (width 0) (type default))
-  )
-  (wire (pts (xy 166.37 121.92) (xy 173.99 121.92))
-    (stroke (width 0) (type default))
-  )
-  (wire (pts (xy 166.37 143.51) (xy 173.99 143.51))
     (stroke (width 0) (type default))
   )
@@
     )
   )
+  (symbol (lib_id "Connector:TestPoint_Probe") (at 212.09 138.43 0) (mirror y) (unit 1)
+    (in_bom yes) (on_board yes) (dnp no)
+    (property "Reference" "TP1" (at 205.74 135.89 0)
+      (effects (font (size 1.27 1.27)))
+    )
+    (property "Value" "TestPoint_Probe" (at 199.39 138.7475 0)
+      (effects (font (size 1.27 1.27)) hide)
+    )
+    (property "Footprint" "TestPoint:TestPoint_Pad_D1.5mm" (at 207.01 138.43 0)
+      (effects (font (size 1.27 1.27)) hide)
+    )
+    (property "Datasheet" "~" (at 207.01 138.43 0)
+      (effects (font (size 1.27 1.27)) hide)
+    )
+    (pin "1")
+    (instances
+      (project "vb125_eth_fdcan_pro"
+        (path "/b473bccb-f14c-41d5-b473-137d3ef8ae1e/c16e79c7-955f-4686-8fe9-acff02e57751"
+          (reference "TP1") (unit 1)
+        )
+        (path "/b473bccb-f14c-41d5-b473-137d3ef8ae1e/13d04be1-6d05-4847-9c03-a8fbeeb3fd19"
+          (reference "TP6") (unit 1)
+        )
+        (path "/b473bccb-f14c-41d5-b473-137d3ef8ae1e/6eaf8f36-f4c1-413f-846c-b502b7be2b8c"
+          (reference "TP14") (unit 1)
+        )
+        (path "/b473bccb-f14c-41d5-b473-137d3ef8ae1e/96773d61-2940-42cb-9a0c-01cb58b4a4b5"
+          (reference "TP37") (unit 1)
+        )
+        (path "/b473bccb-f14c-41d5-b473-137d3ef8ae1e/1ac386c6-64ba-4865-8e07-7f3718b45cdc"
+          (reference "TP41") (unit 1)
+        )
+        (path "/b473bccb-f14c-41d5-b473-137d3ef8ae1e"
+          (reference "TP37") (unit 1)
+        )
+      )
+    )
+  )
   (sheet (at 217.17 90.17) (size 31.75 7.62) (fields_autoplaced)
     (stroke (width 0.1524) (type solid))
@@
       (effects (font (size 1.27 1.27)) (justify left top))
     )
-    (pin "FDCAN3_RX" input (at 166.37 143.51 0)
-      (effects (font (size 1.27 1.27)) (justify right))
-    )
-    (pin "FDCAN3_TX" output (at 166.37 140.97 0)
-      (effects (font (size 1.27 1.27)) (justify right))
-    )
-    (pin "TERM2_EN" output (at 166.37 147.32 0)
-      (effects (font (size 1.27 1.27)) (justify right))
-    )
-    (pin "TERM2_DIS" output (at 166.37 149.86 0)
-      (effects (font (size 1.27 1.27)) (justify right))
-    )
-    (pin "FDCAN1_RX" input (at 166.37 121.92 0)
-      (effects (font (size 1.27 1.27)) (justify right))
-    )
-    (pin "FDCAN1_TX" output (at 166.37 119.38 0)
-      (effects (font (size 1.27 1.27)) (justify right))
-    )
-    (pin "TERM1_EN" output (at 166.37 125.73 0)
-      (effects (font (size 1.27 1.27)) (justify right))
-    )
-    (pin "TERM1_DIS" output (at 166.37 128.27 0)
-      (effects (font (size 1.27 1.27)) (justify right))
-    )
+    (pin "FDCAN3_RX" input (at 166.37 121.92 0)
+      (effects (font (size 1.27 1.27)) (justify right))
+    )
+    (pin "FDCAN3_TX" output (at 166.37 119.38 0)
+      (effects (font (size 1.27 1.27)) (justify right))
+    )
+    (pin "TERM2_EN" output (at 166.37 125.73 0)
+      (effects (font (size 1.27 1.27)) (justify right))
+    )
+    (pin "TERM2_DIS" output (at 166.37 128.27 0)
+      (effects (font (size 1.27 1.27)) (justify right))
+    )
+    (pin "FDCAN1_RX" input (at 166.37 143.51 0)
+      (effects (font (size 1.27 1.27)) (justify right))
+    )
+    (pin "FDCAN1_TX" output (at 166.37 140.97 0)
+      (effects (font (size 1.27 1.27)) (justify right))
+    )
+    (pin "TERM1_EN" output (at 166.37 147.32 0)
+      (effects (font (size 1.27 1.27)) (justify right))
+    )
+    (pin "TERM1_DIS" output (at 166.37 149.86 0)
+      (effects (font (size 1.27 1.27)) (justify right))
+    )
