File: vb125_eth_fdcan_pro/p4_usb.kicad_sch (KiCad schematic)
At the start: 31 parts, among them J5 USB_C_Receptacle_USB2.0, U3 NCP563SQ18T1G, U4 USB3315, X1 24MHz

Commit message: Update outline.
Parts:
- D2: footprint Diode_SMD:D_SMF -> vhrd_diode:D_SMF
- X1: footprint Oscillator:Oscillator_SMD_Abracon_ASE-4Pin_3.2x2.5mm -> vhrd_crystal:Oscillator_SMD_Abracon_ASE-4Pin_3.2x2.5mm
Changed lines of the file:
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@@
       (effects (font (size 1.27 1.27)) (justify left))
     )
-    (property "Footprint" "Oscillator:Oscillator_SMD_Abracon_ASE-4Pin_3.2x2.5mm" (at 217.17 199.39 0)
+    (property "Footprint" "vhrd_crystal:Oscillator_SMD_Abracon_ASE-4Pin_3.2x2.5mm" (at 217.17 199.39 0)
       (effects (font (size 1.27 1.27)) hide)
     )
@@
       (effects (font (size 1.27 1.27)) (justify left))
     )
-    (property "Footprint" "Diode_SMD:D_SMF" (at 168.91 68.58 0)
-      (effects (font (size 1.27 1.27)) hide)
-    )
+    (property "Footprint" "vhrd_diode:D_SMF" (at 168.91 68.58 0)
+      (effects (font (size 1.27 1.27)) hide)
+    )
