File: vb125_eth_fdcan_pro/p8_poe.kicad_sch (KiCad schematic)
At the start: 58 parts, among them Q5 MMBTA42, Q6 Si3440DV, Q7 2N7002, T1 PA1134NL, U11 LTC4267, U12 PS2911-1-F3-AX, U13 ZR431

Commit message: Finish layout.
Parts:
- removed TP1: TestPoint_Probe, TestPoint:TestPoint_Pad_D1.5mm, symbol Connector:TestPoint_Probe
Changed lines of the file:
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@@
   (junction (at 176.53 160.02) (diameter 0) (color 0 0 0 0)
-  )
-  (junction (at 269.24 82.55) (diameter 0) (color 0 0 0 0)
   )
   (junction (at 287.02 129.54) (diameter 0) (color 0 0 0 0)
@@
   )
   (wire (pts (xy 227.33 146.05) (xy 227.33 170.18))
-    (stroke (width 0) (type default))
-  )
-  (wire (pts (xy 269.24 80.01) (xy 269.24 82.55))
     (stroke (width 0) (type default))
   )
@@
         )
       )
-    )
-  )
-  (symbol (lib_id "Connector:TestPoint_Probe") (at 269.24 80.01 0) (mirror y) (unit 1)
-    (in_bom yes) (on_board yes) (dnp no)
-    (property "Reference" "TP1" (at 262.89 77.47 0)
-      (effects (font (size 1.27 1.27)))
-    )
-    (property "Value" "TestPoint_Probe" (at 256.54 80.3275 0)
-      (effects (font (size 1.27 1.27)) hide)
-    )
-    (property "Footprint" "TestPoint:TestPoint_Pad_D1.5mm" (at 264.16 80.01 0)
-      (effects (font (size 1.27 1.27)) hide)
-    )
-    (property "Datasheet" "~" (at 264.16 80.01 0)
-      (effects (font (size 1.27 1.27)) hide)
-    )
-    (pin "1")
-    (instances
-      (project "vb125_eth_fdcan_pro"
-        (path "/b473bccb-f14c-41d5-b473-137d3ef8ae1e/c16e79c7-955f-4686-8fe9-acff02e57751"
-          (reference "TP1") (unit 1)
-        )
-        (path "/b473bccb-f14c-41d5-b473-137d3ef8ae1e/13d04be1-6d05-4847-9c03-a8fbeeb3fd19"
-          (reference "TP6") (unit 1)
-        )
-        (path "/b473bccb-f14c-41d5-b473-137d3ef8ae1e/6eaf8f36-f4c1-413f-846c-b502b7be2b8c"
-          (reference "TP14") (unit 1)
-        )
-        (path "/b473bccb-f14c-41d5-b473-137d3ef8ae1e/5caca214-bd98-4d53-9e0b-a904082b09c6"
-          (reference "TP30") (unit 1)
-        )
-      )

Commit message: Update sch and pcb.
Parts:
- removed C103: Y rated, SMD 1808, vhrd_generic:C_1808_4520Metric, symbol Device:C
- C101: footprint Capacitor_THT:C_Disc_D7.0mm_W2.5mm_P5.00mm -> vhrd_generic:C_Disc_D7.0mm_W2.5mm_P6.00mm; now fitted; now in the parts list
Changed lines of the file:
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@@
   (junction (at 163.83 110.49) (diameter 0) (color 0 0 0 0)
   )
-  (junction (at 265.43 195.58) (diameter 0) (color 0 0 0 0)
-  )
   (junction (at 285.75 114.3) (diameter 0) (color 0 0 0 0)
   )
@@
   )
   (junction (at 140.97 160.02) (diameter 0) (color 0 0 0 0)
-  )
-  (junction (at 293.37 195.58) (diameter 0) (color 0 0 0 0)
   )
   (junction (at 218.44 60.96) (diameter 0) (color 0 0 0 0)
@@
     (stroke (width 0) (type default))
   )
-  (wire (pts (xy 293.37 204.47) (xy 293.37 195.58))
+  (wire (pts (xy 293.37 190.5) (xy 293.37 204.47))
     (stroke (width 0) (type default))
   )
@@
     (stroke (width 0) (type default))
   )
-  (wire (pts (xy 265.43 204.47) (xy 265.43 195.58))
+  (wire (pts (xy 265.43 190.5) (xy 265.43 204.47))
     (stroke (width 0) (type default))
   )
@@
   )
   (wire (pts (xy 284.48 127) (xy 287.02 127))
-    (stroke (width 0) (type default))
-  )
-  (wire (pts (xy 293.37 195.58) (xy 293.37 190.5))
     (stroke (width 0) (type default))
   )
@@
     (stroke (width 0) (type default))
   )
-  (wire (pts (xy 265.43 195.58) (xy 265.43 190.5))
-    (stroke (width 0) (type default))
-  )
   (wire (pts (xy 156.21 60.96) (xy 156.21 110.49))
     (stroke (width 0) (type default))
@@
     (stroke (width 0) (type default))
   )
-  (wire (pts (xy 283.21 195.58) (xy 293.37 195.58))
-    (stroke (width 0) (type default))
-  )
   (wire (pts (xy 128.27 160.02) (xy 115.57 160.02))
     (stroke (width 0) (type default))
@@
   )
   (wire (pts (xy 176.53 130.81) (xy 176.53 160.02))
-    (stroke (width 0) (type default))
-  )
-  (wire (pts (xy 265.43 195.58) (xy 275.59 195.58))
     (stroke (width 0) (type default))
   )
@@
     )
   )
-  (symbol (lib_id "Device:C") (at 279.4 195.58 90) (mirror x) (unit 1)
-    (in_bom yes) (on_board yes) (dnp no)
-    (property "Reference" "C103" (at 278.13 199.39 90)
-      (effects (font (size 1.27 1.27)) (justify left))
-    )
-    (property "Value" "Y rated, SMD 1808" (at 273.05 201.93 90)
-      (effects (font (size 1.27 1.27)) (justify right))
-    )
-    (property "Footprint" "vhrd_generic:C_1808_4520Metric" (at 283.21 196.5452 0)
-      (effects (font (size 1.27 1.27)) hide)
-    )
-    (property "Datasheet" "~" (at 279.4 195.58 0)
-      (effects (font (size 1.27 1.27)) hide)
-    )
-    (property "Variant" "poe" (at 279.4 195.58 0)
-      (effects (font (size 1.27 1.27)) hide)
-    )
-    (pin "1")
-    (pin "2")
-    (instances
-      (project "vb125_eth_fdcan_pro"
-        (path "/b473bccb-f14c-41d5-b473-137d3ef8ae1e/96773d61-2940-42cb-9a0c-01cb58b4a4b5"
-          (reference "C103") (unit 1)
-        )
-        (path "/b473bccb-f14c-41d5-b473-137d3ef8ae1e/1ac386c6-64ba-4865-8e07-7f3718b45cdc"
-          (reference "C104") (unit 1)
-        )
-        (path "/b473bccb-f14c-41d5-b473-137d3ef8ae1e/5caca214-bd98-4d53-9e0b-a904082b09c6"
-          (reference "C93") (unit 1)
-        )
-      )
-    )
-  )
   (symbol (lib_id "Device:C") (at 220.98 96.52 0) (unit 1)
     (in_bom yes) (on_board yes) (dnp no)
@@
   )
   (symbol (lib_id "Device:C") (at 279.4 190.5 90) (unit 1)
-    (in_bom no) (on_board yes) (dnp yes) (fields_autoplaced)
+    (in_bom yes) (on_board yes) (dnp no) (fields_autoplaced)
     (property "Reference" "C101" (at 273.4321 184.15 90)
       (effects (font (size 1.27 1.27)) (justify right))
@@
       (effects (font (size 1.27 1.27)) (justify left))
     )
-    (property "Footprint" "Capacitor_THT:C_Disc_D7.0mm_W2.5mm_P5.00mm" (at 283.21 189.5348 0)
-      (effects (font (size 1.27 1.27)) hide)
-    )
+    (property "Footprint" "vhrd_generic:C_Disc_D7.0mm_W2.5mm_P6.00mm" (at 283.21 189.5348 0)
+      (effects (font (size 1.27 1.27)) hide)
+    )

Commit message: Update outline.
Parts:
- D11: footprint Diode_SMD:D_SMA -> vhrd_diode:D_SMA
- D12: footprint Diode_SMD:D_SOD-323 -> vhrd_diode:D_SOD-323
- D13, D14, D15: footprint Diode_SMD:D_SOD-523 -> vhrd_diode:D_SOD-523
Changed lines of the file:
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@@
       (effects (font (size 1.27 1.27)))
     )
-    (property "Footprint" "Diode_SMD:D_SOD-523" (at 254 128.905 0)
+    (property "Footprint" "vhrd_diode:D_SOD-523" (at 254 128.905 0)
       (effects (font (size 1.27 1.27)) hide)
     )
@@
       (effects (font (size 1.27 1.27)) (justify right))
     )
-    (property "Footprint" "Diode_SMD:D_SOD-523" (at 271.145 148.59 0)
+    (property "Footprint" "vhrd_diode:D_SOD-523" (at 271.145 148.59 0)
       (effects (font (size 1.27 1.27)) hide)
     )
@@
       (effects (font (size 1.27 1.27)))
     )
-    (property "Footprint" "Diode_SMD:D_SOD-523" (at 254 161.925 0)
+    (property "Footprint" "vhrd_diode:D_SOD-523" (at 254 161.925 0)
       (effects (font (size 1.27 1.27)) hide)
     )
@@
       (effects (font (size 1.27 1.27)) (justify left))
     )
-    (property "Footprint" "Diode_SMD:D_SMA" (at 140.97 127 0)
+    (property "Footprint" "vhrd_diode:D_SMA" (at 140.97 127 0)
       (effects (font (size 1.27 1.27)) hide)
     )
@@
       (effects (font (size 1.27 1.27)))
     )
-    (property "Footprint" "Diode_SMD:D_SOD-323" (at 187.96 88.9 0)
-      (effects (font (size 1.27 1.27)) hide)
-    )
+    (property "Footprint" "vhrd_diode:D_SOD-323" (at 187.96 88.9 0)
+      (effects (font (size 1.27 1.27)) hide)
+    )
