File: vb125_eth_fdcan_pro/p6_can_ch1.kicad_sch (KiCad schematic)
At the start: 35 parts, among them J6 D09P33E4GL00LF, K1 EE2-4.5TNUH, M2 B0505MT-1WR4, Q1 BSS138, U7 ADM3050EBRIZ, U8 TLP2270

Commit message: Floorplan work.
Connections:
- net +5V0_MFLT: now reaches C1.1, L3.2, M2.13 (VIN), M2.14 (VIN)
Changed lines of the file:
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@@
+    (effects (font (size 1.27 1.27)) (justify left bottom))
+  )
+  (label "+5V0_MFLT" (at 158.75 72.39 0) (fields_autoplaced)
     (effects (font (size 1.27 1.27)) (justify left bottom))
   )

Commit message: Finish layout.
Parts:
- added E1, E3, E5: SparkGap, symbol Device:SparkGap
Connections:
- net +VIN_DB9: now also E5.2; no longer J6.1
- net CAN_H: now also K1.5, E1.2; no longer R19.1
- net CAN_L: now also K1.8, E3.2; no longer R19.1
- net CHASSIS: now also E1.1, E3.1, E5.1
- net at R19.2: now also C36.1, R19.2; no longer K1.5
- new net: K1.4, R19.1
- new net: K1.9, R19.1
- no-connect marks 5 -> 6
Other:
- moved on the sheet: C36, J6, R19

Commit message: Update sch and pcb.
Parts:
- removed C66: Y rated, SMD 1808, vhrd_generic:C_1808_4520Metric, symbol Device:C
- removed E5: SparkGap, symbol Device:SparkGap
- added JP1: SolderJumper_2_Open, Jumper:SolderJumper-2_P1.3mm_Open_RoundedPad1.0x1.5mm, symbol Jumper:SolderJumper_2_Open
- C65: footprint Capacitor_THT:C_Disc_D7.0mm_W2.5mm_P5.00mm -> vhrd_generic:C_Disc_D7.0mm_W2.5mm_P6.00mm; now fitted; now in the parts list
- E1, E3: footprint (none) -> vhrd_generic:SPARK_GAP_011
Connections:
- net CAN_H: now also E1.1; no longer E1.2
- net CAN_L: now also E3.1; no longer E3.2
- net CHASSIS: now also E1.2, E3.2, JP1.1 (A); no longer E1.1, E3.1
- net at J6.5: now also JP1.2 (B)
- no-connect marks 6 -> 5
Other:
- note added: "CiA DS102: 1: RSVD 2: CAN_L 3: CAN_GND 4: RSVD 5: CAN_SHLD (optional) 6: CAN_GND (optional) 7: CAN_H 8: RSVD (error line) 9: CAN_V+ (optional, txvs and optocouplers)"
- moved on the sheet: E1, E3, J6

Commit message: Update outline.
Parts:
- D12: footprint Diode_SMD:D_SOD-523 -> vhrd_diode:D_SOD-523
Changed lines of the file:
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@@
       (effects (font (size 1.27 1.27)))
     )
-    (property "Footprint" "Diode_SMD:D_SOD-523" (at 271.145 157.48 0)
+    (property "Footprint" "vhrd_diode:D_SOD-523" (at 271.145 157.48 0)
       (effects (font (size 1.27 1.27)) hide)
     )
@@
       (effects (font (size 1.27 1.27)))
     )
-    (property "Footprint" "Diode_SMD:D_SOD-523" (at 231.775 157.48 0)
-      (effects (font (size 1.27 1.27)) hide)
-    )
+    (property "Footprint" "vhrd_diode:D_SOD-523" (at 231.775 157.48 0)
+      (effects (font (size 1.27 1.27)) hide)
+    )
